Commit message: Extract void frontier

File: config/baxter_yyj.urdf (robot description, URDF)
Before this commit: robot baxter, 50 links, 49 joints
Links:
- link camera_rgb_optical_frame: geometry collision box size=0.22 0.03 0.035; visual box size=0.2 0.03 0.035
Joints:
- joint camera_rgb_optical_frame: origin xyz=0.000324725 -0.09238 0.0204097 rpy=0.0745256 0.0039322 0.129185 -> xyz=-0.00139927 -0.0843446 0.0143339 rpy=0.0758307 0.00234285 0.13389

Commit message: Remove the redundant code

File: config/baxter_yyj.urdf (robot description, URDF)
Before this commit: robot baxter, 50 links, 49 joints
Links:
- link right_lower_shoulder: geometry collision cylinder length=0.22 radius=0.08; visual mesh filename=package://baxter_description/meshes/lower_shoulder/S1.DAE
Joints:
- joint camera_rgb_optical_frame: origin xyz=-0.00139927 -0.0843446 0.0143339 rpy=0.0758307 0.00234285 0.13389 -> xyz=-0.0100727 -0.0809104 0.0183719 rpy=0.136204 0.013331 0.0674753

Commit message: Add a new exploration strategy based on weighted continuity score and information gain score

File: config/baxter_yyj.urdf (robot description, URDF)
Before this commit: robot baxter, 50 links, 49 joints
Links:
- link left_upper_shoulder: geometry collision cylinder length=0.2722 radius=0.08; visual mesh filename=package://baxter_description/meshes/upper_shoulder/S0.DAE
- link right_lower_shoulder: geometry collision cylinder length=0.25 radius=0.15; visual mesh filename=package://baxter_description/meshes/lower_shoulder/S1.DAE
- link right_upper_shoulder: geometry collision cylinder length=0.43 radius=0.08; visual mesh filename=package://baxter_description/meshes/upper_shoulder/S0.DAE
Joints:
- joint camera_rgb_optical_frame: origin xyz=-0.0100727 -0.0809104 0.0183719 rpy=0.136204 0.013331 0.0674753 -> xyz=-0.00485757 -0.0810587 0.0164881 rpy=0.178573 -0.00506743 0.0677429

Commit message: Some modifications in order to explore completely

File: config/baxter_yyj.urdf (robot description, URDF)
Before this commit: robot baxter, 50 links, 49 joints
Joints:
- joint camera_rgb_optical_frame: origin xyz=-0.00485757 -0.0810587 0.0164881 rpy=0.178573 -0.00506743 0.0677429 -> xyz=-0.00816875 -0.0701083 0.0151665 rpy=0.316951 -0.0163395 0.0607724
